File: Hardware-TinyPicoLoraGateway.kicad_sch (KiCad schematic)
At the start: 15 parts

Commit message: Update 2023-01-25
Parts:
- removed C? (x2): 0.1u, symbol Device:C_Small
- removed J?: Antenna_Hole, symbol Connector:Conn_01x01_Male
- removed J?: Conn_01x05_Female, symbol Connector:Conn_01x05_Female
- removed J?: GroundHole(dipole), symbol Connector:Conn_01x01_Male
- removed R? (x2): 10k, symbol Device:R_Small
- removed R? (x2): 30, symbol Device:R_Small
- removed R?: 100, symbol Device:R_Small
- removed U?: 74LVC1G14, symbol 74xGxx:74LVC1G14
- removed U?: TinyPico, symbol dmc_dev_modules:TinyPico
- added J1: SMA, Connector_Coaxial:SMA_Amphenol_132289_EdgeMount, symbol Connector:Conn_Coaxial
- added J2: Antenna_Hole, Connector_PinHeader_2.54mm:PinHeader_1x01_P2.54mm_Vertical, symbol Connector:Conn_01x01_Male
- added J3: U.fl, Connector_Coaxial:U.FL_Hirose_U.FL-R-SMT-1_Vertical, symbol Connector:Conn_Coaxial
- added U1: UM_Tiny_ESP32_S3, UnexpectedMaker-ESP32S3:TinyS3, symbol dmc_dev_modules:UM_Tiny_ESP32_S3
- C3: renamed from C?; footprint (none) -> Capacitor_SMD:C_1206_3216Metric; LCSC Part (none) -> C110253
- C5: renamed from C?; footprint (none) -> Capacitor_Tantalum_SMD:CP_EIA-3216-18_Kemet-A; LCSC Part (none) -> C7177
- U4: renamed from U?; footprint (none) -> RF_Module:HOPERF_RFM9XW_SMD
Connections:
- net +3.3V: now also U1.4 (3V3)
- net GND: now also J1.2 (Ext), J3.2 (Ext), U1.14 (GND), U1.2 (GND)
- net RFM95_DIO0: now also U1.20 (IO34)
- net RFM95_NSS: now also U1.7 (IO3)
- net RFM95_RST: now also U1.19 (IO9-SCL)
- net RFM95_DIO3: now reaches U4.11 (DIO3)
- net RFM95_DIO3: now also U1.16 (IO6)
- net RFM95_DIO4: now reaches U4.12 (DIO4)
- net RFM95_DIO4: now also U1.18 (IO8-SDA)
- net RFM95_DIO1: now reaches U4.15 (DIO1)
- net RFM95_DIO1: now also U1.9 (IO5)
- net RFM95_DIO2: now reaches U4.16 (DIO2)
- net RFM95_DIO2: now also U1.8 (IO4)
- net RFM95_DIO5: now reaches U4.7 (DIO5)
- net RFM95_DIO5: now also U1.17 (IO7)
- net at U4.9 (ANT): now also J1.1 (In), J2.1 (Pin_1), J3.1 (In)
- net RFM95_MISO renamed MISO
- net MISO: now also U1.22 (IO37-MI)
- net RFM95_MOSI renamed MOSI
- net MOSI: now also U1.23 (IO35-MO)
- net RFM95_SCK renamed SCK
- net SCK: now also U1.21 (IO36-SCK)
- no-connect marks 12 -> 8
Other:
- note added: "RFM 95 LoRa"
- moved on the sheet: C3, C5, U4
